File: Placa_de_Iluminação_Weiss/Placa_de_Iluminação_Weiss.kicad_sch (KiCad schematic)
At the start: 6 parts

Commit message: feat: README da placa de processamento do foguete Weiss adicionado
Connections:
- net +3.3V: no longer SW1.3 (K)
- net at R2.1: now also SW1.3 (K); no longer SW1.2
- net at SW1.1: no longer R1.1
- new net: R1.1, SW1.2
Changed lines of the file:
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@@
 	(paper "A4")
-	(junction
-		(at 203.2 91.44)
-		(diameter 0)
-		(color 0 0 0 0)
-	)
 	(junction
 		(at 222.25 92.71)
@@
 	(wire
 		(pts
-			(xy 193.04 91.44) (xy 193.04 88.9)
+			(xy 203.2 91.44) (xy 210.82 91.44)
 		)
 		(stroke
@@
 	(wire
 		(pts
-			(xy 203.2 91.44) (xy 210.82 91.44)
+			(xy 187.96 88.9) (xy 187.96 93.98)
 		)
 		(stroke
@@
 	(wire
 		(pts
+			(xy 193.04 93.98) (xy 187.96 93.98)
+		)
+		(stroke
+			(width 0)
+			(type default)
+		)
+	)
+	(wire
+		(pts
 			(xy 219.71 88.9) (xy 219.71 91.44)
 		)
@@
 			(type default)
 			(color 0 0 0 1)
+		)
+	)
+	(wire
+		(pts
+			(xy 203.2 93.98) (xy 203.2 99.06)
+		)
+		(stroke
+			(width 0)
+			(type default)
 		)
 	)
@@
 	(wire
 		(pts
-			(xy 193.04 99.06) (xy 187.96 99.06)
+			(xy 187.96 99.06) (xy 203.2 99.06)
 		)
 		(stroke
@@
 	(wire
 		(pts
-			(xy 193.04 93.98) (xy 193.04 99.06)
-		)
-		(stroke
-			(width 0)
-			(type default)
-		)
-	)
-	(wire
-		(pts
 			(xy 180.34 88.9) (xy 176.53 88.9)
 		)
 		(stroke
-			(width 0)
-			(type default)
-		)
-	)
-	(wire
-		(pts
-			(xy 193.04 88.9) (xy 187.96 88.9)
-		)
-		(stroke
-			(width 0)
-			(type default)
-		)
-	)
-	(wire
-		(pts
-			(xy 203.2 91.44) (xy 203.2 93.98)
-		)
-		(stroke
