File: placa_de_telemetria_weiss/Receptor Solo.brd (EAGLE design)
At the start: 61.9 x 84.3 mm, 6 parts

Commit message: Atualização da placa de telemetria
Routing:
- net GND: track 97.0 -> 0.00 mm, vias 2 -> 0
- net N$1: track 55.9 -> 51.5 mm
- net N$4: track 59.3 -> 57.3 mm
- net N$2: track 57.0 -> 55.2 mm
- net N$3: track 59.3 -> 57.7 mm
- net VCC: track 14.7 -> 15.2 mm
Changed lines of the file:
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@@
 <contactref element="U$2" pad="M0"/>
 <wire x1="32.167" y1="68.948" x2="32.245" y2="68.87" width="1.7" layer="16"/>
-<wire x1="45.5066" y1="60.3897875" x2="45.5066" y2="45.5494" width="1.7" layer="16"/>
-<wire x1="45.5066" y1="45.5494" x2="41.7958" y2="41.8386" width="1.7" layer="16"/>
-<wire x1="32.245" y1="68.87" x2="37.0263875" y2="68.87" width="1.7" layer="16"/>
-<wire x1="37.0263875" y1="68.87" x2="45.5066" y2="60.3897875" width="1.7" layer="16"/>
-<wire x1="46.3672" y1="33.04" x2="54.63" y2="33.04" width="1.7" layer="16"/>
-<wire x1="41.7958" y1="41.8386" x2="41.7958" y2="37.6114" width="1.7" layer="16"/>
-<wire x1="41.7958" y1="37.6114" x2="46.3672" y2="33.04" width="1.7" layer="16"/>
+<wire x1="44.786" y1="62.5094" x2="44.786" y2="38.3" width="1.7" layer="16"/>
+<wire x1="32.245" y1="68.87" x2="38.4254" y2="68.87" width="1.7" layer="16"/>
+<wire x1="38.4254" y1="68.87" x2="44.786" y2="62.5094" width="1.7" layer="16"/>
+<wire x1="44.786" y1="38.3" x2="50.046" y2="33.04" width="1.7" layer="16"/>
+<wire x1="50.046" y1="33.04" x2="54.63" y2="33.04" width="1.7" layer="16"/>
 </signal>
 <signal name="N$2">
@@
 <contactref element="U$2" pad="M1"/>
 <wire x1="32.167" y1="66.408" x2="32.245" y2="66.33" width="1.7" layer="16"/>
-<wire x1="39.3338" y1="42.8584" x2="39.3338" y2="36.5916" width="1.7" layer="16"/>
-<wire x1="43.0446" y1="59.3699875" x2="43.0446" y2="46.5692" width="1.7" layer="16"/>
-<wire x1="43.0446" y1="46.5692" x2="39.3338" y2="42.8584" width="1.7" layer="16"/>
-<wire x1="32.245" y1="66.33" x2="36.0845875" y2="66.33" width="1.7" layer="16"/>
-<wire x1="36.0845875" y1="66.33" x2="43.0446" y2="59.3699875" width="1.7" layer="16"/>
-<wire x1="39.3338" y1="36.5916" x2="47.9654" y2="27.96" width="1.7" layer="16"/>
-<wire x1="47.9654" y1="27.96" x2="54.63" y2="27.96" width="1.7" layer="16"/>
+<wire x1="42.324" y1="61.4896" x2="42.324" y2="32.7896" width="1.7" layer="16"/>
+<wire x1="32.245" y1="66.33" x2="37.4836" y2="66.33" width="1.7" layer="16"/>
+<wire x1="37.4836" y1="66.33" x2="42.324" y2="61.4896" width="1.7" layer="16"/>
+<wire x1="47.1536" y1="27.96" x2="54.63" y2="27.96" width="1.7" layer="16"/>
+<wire x1="42.324" y1="32.7896" x2="47.1536" y2="27.96" width="1.7" layer="16"/>
 </signal>
 <signal name="N$3">
 <contactref element="U$1" pad="GPIO17"/>
 <contactref element="U$2" pad="RXD"/>
+<wire x1="36.5418" y1="63.79" x2="39.862" y2="60.4698" width="1.7" layer="16"/>
+<wire x1="39.862" y1="60.4698" x2="39.862" y2="31.7698" width="1.7" layer="16"/>
 <wire x1="32.167" y1="63.868" x2="32.245" y2="63.79" width="1.7" layer="16"/>
-<wire x1="40.5826" y1="58.3501875" x2="40.5826" y2="47.589" width="1.7" layer="16"/>
-<wire x1="40.5826" y1="47.589" x2="36.8718" y2="43.8782" width="1.7" layer="16"/>
-<wire x1="36.8718" y1="43.8782" x2="36.8718" y2="35.5718" width="1.7" layer="16"/>
-<wire x1="32.245" y1="63.79" x2="35.1427875" y2="63.79" width="1.7" layer="16"/>
-<wire x1="35.1427875" y1="63.79" x2="40.5826" y2="58.3501875" width="1.7" layer="16"/>
-<wire x1="36.8718" y1="35.5718" x2="52.1816" y2="20.262" width="1.7" layer="16"/>
-<wire x1="52.1816" y1="20.262" x2="54.8" y2="20.262" width="1.7" layer="16"/>
-<wire x1="54.8" y1="20.262" x2="54.63" y2="20.34" width="0" layer="19" extent="16-16"/>
+<wire x1="32.245" y1="63.79" x2="36.5418" y2="63.79" width="1.7" layer="16"/>
+<wire x1="51.3698" y1="20.262" x2="54.8" y2="20.262" width="1.7" layer="16"/>
+<wire x1="54.8" y1="20.262" x2="54.722" y2="20.34" width="1.7" layer="16"/>
+<wire x1="54.722" y1="20.34" x2="54.63" y2="20.34" width="1.7" layer="16"/>
+<wire x1="39.862" y1="31.7698" x2="51.3698" y2="20.262" width="1.7" layer="16"/>
 </signal>
 <signal name="N$4">
 <contactref element="U$1" pad="GPIO16"/>
 <contactref element="U$2" pad="TXD"/>
-<wire x1="32.167" y1="61.328" x2="32.245" y2="61.25" width="1.7" layer="16"/>
-<wire x1="38.1206" y1="48.6088" x2="34.1118" y2="44.6" width="1.7" layer="16"/>
-<wire x1="34.1118" y1="44.6" x2="34.1118" y2="34.85" width="1.7" layer="16"/>
-<wire x1="32.245" y1="61.25" x2="34.2009875" y2="61.25" width="1.7" layer="16"/>
-<wire x1="34.2009875" y1="61.25" x2="38.1206" y2="57.3303875" width="1.7" layer="16"/>
-<wire x1="38.1206" y1="57.3303875" x2="38.1206" y2="48.6088" width="1.7" layer="16"/>
-<wire x1="34.1118" y1="34.85" x2="51.1618" y2="17.8" width="1.7" layer="16"/>
-<wire x1="51.1618" y1="17.8" x2="54.63" y2="17.8" width="1.7" layer="16"/>
+<wire x1="32.167" y1="61.328" x2="35.522" y2="61.328" width="1.7" layer="16"/>
+<wire x1="37.4" y1="59.45" x2="37.4" y2="30.75" width="1.7" layer="16"/>
+<wire x1="37.4" y1="30.75" x2="50.35" y2="17.8" width="1.7" layer="16"/>
+<wire x1="50.35" y1="17.8" x2="54.63" y2="17.8" width="1.7" layer="16"/>
+<wire x1="35.522" y1="61.328" x2="37.4" y2="59.45" width="1.7" layer="16"/>
 </signal>
 <signal name="N$5">
@@
 <contactref element="U$2" pad="GND"/>
 <contactref element="LED2" pad="K"/>
-<wire x1="22.22" y1="48.5" x2="27.428" y2="53.708" width="1.7" layer="16"/>
-<wire x1="27.428" y1="53.708" x2="32.167" y2="53.708" width="1.7" layer="16"/>
-<wire x1="22.22" y1="48.5" x2="22.22" y2="48.38" width="1.7" layer="16"/>
-<wire x1="22.22" y1="48.38" x2="25.35" y2="45.25" width="1.7" layer="16"/>
-<wire x1="25.35" y1="45.25" x2="25.35" y2="42.23" width="1.7" layer="16"/>
-<wire x1="22.4009" y1="39.2809" x2="25.35" y2="42.23" width="1.7" layer="16"/>
-<wire x1="25.4" y1="36.12" x2="22.32" y2="39.2" width="1.7" layer="16"/>
-<wire x1="31.77" y1="12.72" x2="31.03" y2="12.72" width="1.7" layer="16"/>
-<wire x1="25.4" y1="18.35" x2="25.4" y2="36.12" width="1.7" layer="16"/>
-<wire x1="31.77" y1="12.72" x2="26.28" y2="12.72" width="1.7" layer="16"/>
-<wire x1="26.28" y1="12.72" x2="24.1" y2="14.9" width="1.7" layer="16"/>
-<wire x1="24.1" y1="14.9" x2="24.1" y2="17.05" width="1.7" layer="16"/>
-<wire x1="24.1" y1="17.05" x2="25.4" y2="18.35" width="1.7" layer="16"/>
-<wire x1="31.77" y1="12.72" x2="41.77" y2="12.72" width="1.7" layer="1"/>
-<wire x1="41.77" y1="12.72" x2="52.339" y2="23.289" width="1.7" layer="1"/>
-<wire x1="52.339" y1="23.289" x2="52.339" y2="24.861" width="1.7" layer="1"/>
-<wire x1="52.339" y1="24.861" x2="52.3" y2="24.9" width="1.7" layer="1"/>
-<via x="52.3" y="24.9" extent="1-16" drill="1"/>
-<wire x1="52.3" y1="24.9" x2="51.0254" y2="24.9" width="1.7" layer="16"/>
-<wire x1="51.0254" y1="24.9" x2="50.4274" y2="25.498" width="1.7" layer="16"/>
-<wire x1="52.3" y1="24.9" x2="52.3" y2="30.5268" width="1.7" layer="1"/>
-<wire x1="52.3" y1="30.5268" x2="52.25" y2="30.5768" width="1.7" layer="1"/>
-<via x="52.25" y="30.5768" extent="1-16" drill="1"/>
-<wire x1="52.25" y1="30.5768" x2="52.2232" y2="30.55" width="1.7" layer="16"/>
-<wire x1="52.2232" y1="30.55" x2="48.9" y2="30.55" width="1.7" layer="16"/>
 <polygon width="1.7" layer="16">
-<vertex x="-15.55" y="107.2"/>
-<vertex x="-15.55" y="-22.9"/>
-<vertex x="117.15" y="-22.9"/>
-<vertex x="117.15" y="107.2"/>
+<vertex x="78.85" y="-5.15"/>
+<vertex x="79.05" y="-5.35"/>
+<vertex x="79.05" y="83.7"/>
+<vertex x="79.45" y="84.1"/>
+<vertex x="12.6" y="84.1"/>
+<vertex x="12.6" y="52.75"/>
+<vertex x="13.3" y="-5.05"/>
 </polygon>
 </signal>
@@
 <contactref element="R1" pad="1"/>
 <contactref element="LED1" pad="A"/>
-<wire x1="20.5234" y1="55.82006875" x2="20.5234" y2="50.10890625" width="1.7" layer="16"/>
-<wire x1="20.5234" y1="50.10890625" x2="19.8868" y2="49.47230625" width="1.7" layer="16"/>
-<wire x1="19.8868" y1="49.47230625" x2="19.8868" y2="48.7068" width="1.7" layer="16"/>
-<wire x1="19.8868" y1="48.7068" x2="19.68" y2="48.5" width="1.7" layer="16"/>
+<wire x1="19.68" y1="48.5" x2="19.68" y2="54.97666875" width="1.7" layer="16"/>
+<wire x1="19.68" y1="54.97666875" x2="20.5234" y2="55.82006875" width="1.7" layer="16"/>
 </signal>
 <signal name="VCC">
 <contactref element="U$1" pad="3.3V"/>
 <contactref element="U$2" pad="VCC"/>
-<wire x1="32.167" y1="56.248" x2="32.245" y2="56.17" width="1.7" layer="16"/>
-<wire x1="32.245" y1="56.17" x2="34.2009875" y2="56.17" width="1.7" layer="16"/>
-<wire x1="34.2009875" y1="56.17" x2="35.6586" y2="54.7123875" width="1.7" layer="16"/>
-<wire x1="35.6586" y1="54.7123875" x2="35.6586" y2="49.6286" width="1.7" layer="16"/>
-<wire x1="35.6586" y1="49.6286" x2="31.77" y2="45.74" width="1.7" layer="16"/>
+<wire x1="32.167" y1="56.248" x2="32.0518" y2="56.1328" width="1.7" layer="16"/>
+<wire x1="32.0518" y1="56.1328" x2="30.0958125" y2="56.1328" width="1.7" layer="16"/>
+<wire x1="30.0958125" y1="56.1328" x2="28.2" y2="54.2369875" width="1.7" layer="16"/>
+<wire x1="28.2" y1="54.2369875" x2="28.2" y2="48.55" width="1.7" layer="16"/>
+<wire x1="28.2" y1="48.55" x2="31.01" y2="45.74" width="1.7" layer="16"/>
+<wire x1="31.01" y1="45.74" x2="31.77" y2="45.74" width="1.7" layer="16"/>
 </signal>
 <signal name="N$9">
